File: crossover/KiCad/Two_Way_Crossover.sch (KiCad schematic (older format))
At the start: 21 parts, among them J1 Conn_01x01_Female, J2 Conn_01x01_Female, J3 Woofer, J4 Tweeter

Commit message: Redesign PCB
Parts:
- removed R4, R6: 8R2, Resistor_THT:R_Axial_Power_L60.0mm_W14.0mm_P66.04mm, symbol Device:R
- L1, L2, L3: footprint Inductor_THT:L_Radial_D40.6mm_P26.16mm_Vishay_IHB-5 -> etal_Inductors:Radial_D36.5mm_H12.0mm_P23.0mm
- R1, R2: footprint Resistor_THT:R_Axial_Power_L60.0mm_W14.0mm_P66.04mm -> etal_Power_Resistor:Resistor_Power_Axial_L91.5_W20.2_H20.2
- R3: value 8R2 -> 4R7; # Royal Ohm PRW020JW82JB00 -> SR Passives CRL40W-4R7
- R4: renamed from R5; value 8R2 -> 4R7; # Royal Ohm PRW020JW82JB00 -> SR Passives CRL40W-4R7
Other:
- moved on the sheet: R4
Changed lines of the file:
@@
 EESchema Schematic File Version 4
-LIBS:Two_Way_Crossover-cache
 EELAYER 30 0
 EELAYER END
@@
 F 0 "L1" V 1590 1350 50  0000 C CNN
 F 1 "1m" V 1499 1350 50  0000 C CNN
-F 2 "Inductor_THT:L_Radial_D40.6mm_P26.16mm_Vishay_IHB-5" H 1400 1350 50  0001 C CNN
+F 2 "etal_Inductors:Radial_D36.5mm_H12.0mm_P23.0mm" H 1400 1350 50  0001 C CNN
 F 3 "https://www.tme.eu/Document/df8507a2705344364f8bbbdd89330ed2/VISATON-SP.pdf" H 1400 1350 50  0001 C CNN
 F 4 "Visaton 4986" V 1400 1350 50  0001 C CNN "#"
@@
 F 0 "L2" H 1702 3396 50  0000 L CNN
 F 1 "m47" H 1702 3305 50  0000 L CNN
-F 2 "Inductor_THT:L_Radial_D40.6mm_P26.16mm_Vishay_IHB-5" H 1650 3350 50  0001 C CNN
+F 2 "etal_Inductors:Radial_D36.5mm_H12.0mm_P23.0mm" H 1650 3350 50  0001 C CNN
 F 3 "https://www.tme.eu/Document/df8507a2705344364f8bbbdd89330ed2/VISATON-SP.pdf" H 1650 3350 50  0001 C CNN
 F 4 "Visaton 4993" H 1650 3350 50  0001 C CNN "#"
@@
 F 0 "R1" V 1943 1500 50  0000 C CNN
 F 1 "8R2" V 2034 1500 50  0000 C CNN
-F 2 "Resistor_THT:R_Axial_Power_L60.0mm_W14.0mm_P66.04mm" V 2080 1500 50  0001 C CNN
+F 2 "etal_Power_Resistor:Resistor_Power_Axial_L91.5_W20.2_H20.2" V 2080 1500 50  0001 C CNN
 F 3 "https://www.tme.eu/Document/27c0719e632264b7132c0e127fb04b62/ax20w.pdf" H 2150 1500 50  0001 C CNN
 F 4 "Royal Ohm PRW020JW82JB00" V 2150 1500 50  0001 C CNN "#"
@@
 F 0 "L3" V 2340 1350 50  0000 C CNN
 F 1 "1m" V 2249 1350 50  0000 C CNN
-F 2 "Inductor_THT:L_Radial_D40.6mm_P26.16mm_Vishay_IHB-5" H 2150 1350 50  0001 C CNN
+F 2 "etal_Inductors:Radial_D36.5mm_H12.0mm_P23.0mm" H 2150 1350 50  0001 C CNN
 F 3 "https://www.tme.eu/Document/df8507a2705344364f8bbbdd89330ed2/VISATON-SP.pdf" H 2150 1350 50  0001 C CNN
 F 4 "Visaton 4986" V 2150 1350 50  0001 C CNN "#"
@@
 $Comp
 L Device:R R4
-U 1 1 5DE2C82E
-P 2300 3100
-F 0 "R4" V 2093 3100 50  0000 C CNN
-F 1 "8R2" V 2184 3100 50  0000 C CNN
-F 2 "Resistor_THT:R_Axial_Power_L60.0mm_W14.0mm_P66.04mm" V 2230 3100 50  0001 C CNN
-F 3 "https://www.tme.eu/Document/27c0719e632264b7132c0e127fb04b62/ax20w.pdf" H 2300 3100 50  0001 C CNN
-F 4 "Royal Ohm PRW020JW82JB00" V 2300 3100 50  0001 C CNN "#"
-	1    2300 3100
-	0    -1   -1   0
-$EndComp
-Wire Wire Line
-	2150 3100 2100 3100
-Wire Wire Line
-	2100 3100 2100 2950
-Wire Wire Line
-	2100 2950 2150 2950
-Wire Wire Line
-	2100 2950 2050 2950
-Connection ~ 2100 2950
-Wire Wire Line
-	2450 3100 2500 3100
-Wire Wire Line
-	2500 3100 2500 2950
-$Comp
-L Device:R R5
 U 1 1 5DE34B39
-P 2500 3500
-F 0 "R5" V 2293 3500 50  0000 C CNN
-F 1 "8R2" V 2384 3500 50  0000 C CNN
-F 2 "Resistor_THT:R_Axial_Power_L60.0mm_W14.0mm_P66.04mm" V 2430 3500 50  0001 C CNN
-F 3 "https://www.tme.eu/Document/27c0719e632264b7132c0e127fb04b62/ax20w.pdf" H 2500 3500 50  0001 C CNN
-F 4 "Royal Ohm PRW020JW82JB00" V 2500 3500 50  0001 C CNN "#"
-	1    2500 3500
-	1    0    0    -1
-$EndComp
-$Comp
-L Device:R R6
-U 1 1 5DE35B56
-P 2650 3500
-F 0 "R6" V 2443 3500 50  0000 C CNN
-F 1 "8R2" V 2534 3500 50  0000 C CNN
-F 2 "Resistor_THT:R_Axial_Power_L60.0mm_W14.0mm_P66.04mm" V 2580 3500 50  0001 C CNN
-F 3 "https://www.tme.eu/Document/27c0719e632264b7132c0e127fb04b62/ax20w.pdf" H 2650 3500 50  0001 C CNN
-F 4 "Royal Ohm PRW020JW82JB00" V 2650 3500 50  0001 C CNN "#"
-	1    2650 3500
-	-1   0    0    1
-$EndComp
-Wire Wire Line
-	2650 3350 2650 3300
-Wire Wire Line
-	2650 3300 2500 3300
-Wire Wire Line
-	2500 3300 2500 3350
-Wire Wire Line
-	2500 3650 2500 3700
-Wire Wire Line
-	2500 3700 2650 3700
-Wire Wire Line
-	2650 3700 2650 3650
-Wire Wire Line
-	2500 3300 2500 3100
-Connection ~ 2500 3100
+P 2500 3300
+F 0 "R4" V 2293 3300 50  0000 C CNN
+F 1 "4R7" V 2384 3300 50  0000 C CNN
+F 2 "Resistor_THT:R_Axial_Power_L60.0mm_W14.0mm_P66.04mm" V 2430 3300 50  0001 C CNN
+F 3 "https://www.tme.eu/Document/d2d66de62be8f045452af502fd3b634f/SR-Passives-CR-W.pdf" H 2500 3300 50  0001 C CNN
+F 4 "SR Passives CRL40W-4R7" V 2500 3300 50  0001 C CNN "#"
+	1    2500 3300
+	1    0    0    -1
+$EndComp
 Wire Wire Line
 	1650 2950 1650 3200
@@
 F 0 "R2" H 2475 1650 50  0000 C CNN
 F 1 "8R2" H 2475 1550 50  0000 C CNN
-F 2 "Resistor_THT:R_Axial_Power_L60.0mm_W14.0mm_P66.04mm" V 2530 1600 50  0001 C CNN
+F 2 "etal_Power_Resistor:Resistor_Power_Axial_L91.5_W20.2_H20.2" V 2530 1600 50  0001 C CNN
 F 3 "https://www.tme.eu/Document/27c0719e632264b7132c0e127fb04b62/ax20w.pdf" H 2600 1600 50  0001 C CNN
 F 4 "Royal Ohm PRW020JW82JB00" V 2600 1600 50  0001 C CNN "#"
@@
 P 2300 2950
 F 0 "R3" V 2093 2950 50  0000 C CNN
-F 1 "8R2" V 2184 2950 50  0000 C CNN
+F 1 "4R7" V 2184 2950 50  0000 C CNN
 F 2 "Resistor_THT:R_Axial_Power_L60.0mm_W14.0mm_P66.04mm" V 2230 2950 50  0001 C CNN
-F 3 "https://www.tme.eu/Document/27c0719e632264b7132c0e127fb04b62/ax20w.pdf" H 2300 2950 50  0001 C CNN
-F 4 "Royal Ohm PRW020JW82JB00" V 2300 2950 50  0001 C CNN "#"
+F 3 "https://www.tme.eu/Document/d2d66de62be8f045452af502fd3b634f/SR-Passives-CR-W.pdf" H 2300 2950 50  0001 C CNN
+F 4 "SR Passives CRL40W-4R7" V 2300 2950 50  0001 C CNN "#"
 	1    2300 2950
 	0    1    1    0
@@
 $EndComp
 Connection ~ 1200 3700
-Wire Wire Line
-	2450 2950 2500 2950
-Connection ~ 2500 2950
-Wire Wire Line
-	2500 2950 3150 2950
-Connection ~ 2500 3300
 $Comp
 L Connector:Screw_Terminal_01x02 J3
@@
 Text Notes 2850 4000 0    59   ~ 0
 High-pass section
+Wire Wire Line
+	2450 2950 2500 2950
+Wire Wire Line
+	2050 2950 2150 2950
+Wire Wire Line
+	2500 3450 2500 3700
+Wire Wire Line
+	2500 3150 2500 2950
+Connection ~ 2500 2950
+Wire Wire Line
+	2500 2950 3150 2950
 $EndSCHEMATC

Commit message: Partially fix incorrect PCB footprints
Parts:
- R1, R2: footprint etal_Power_Resistor:Resistor_Power_Axial_L91.5_W20.2_H20.2 -> Resistor_THT:R_Axial_Power_L60.0mm_W14.0mm_P66.04mm
Changed lines of the file:
@@
 F 0 "R1" V 1943 1500 50  0000 C CNN
 F 1 "8R2" V 2034 1500 50  0000 C CNN
-F 2 "etal_Power_Resistor:Resistor_Power_Axial_L91.5_W20.2_H20.2" V 2080 1500 50  0001 C CNN
+F 2 "Resistor_THT:R_Axial_Power_L60.0mm_W14.0mm_P66.04mm" V 2080 1500 50  0001 C CNN
 F 3 "https://www.tme.eu/Document/27c0719e632264b7132c0e127fb04b62/ax20w.pdf" H 2150 1500 50  0001 C CNN
 F 4 "Royal Ohm PRW020JW82JB00" V 2150 1500 50  0001 C CNN "#"
@@
 F 0 "R2" H 2475 1650 50  0000 C CNN
 F 1 "8R2" H 2475 1550 50  0000 C CNN
-F 2 "etal_Power_Resistor:Resistor_Power_Axial_L91.5_W20.2_H20.2" V 2530 1600 50  0001 C CNN
+F 2 "Resistor_THT:R_Axial_Power_L60.0mm_W14.0mm_P66.04mm" V 2530 1600 50  0001 C CNN
 F 3 "https://www.tme.eu/Document/27c0719e632264b7132c0e127fb04b62/ax20w.pdf" H 2600 1600 50  0001 C CNN
 F 4 "Royal Ohm PRW020JW82JB00" V 2600 1600 50  0001 C CNN "#"

Commit message: Add license
Parts:
- R1, R2: P (none) -> 20W
- R3, R4: footprint Resistor_THT:R_Axial_Power_L60.0mm_W14.0mm_P66.04mm -> etal_Resistors_THT:Resistor_Power_Axial_L91.5_W20.2_H20.2; P (none) -> 40W
Other:
- note added: "Copyright Eero Talus 2020.\n\nThis documentation describes Open Hardware and is licensed under the CERN OHL v. 1.2.\n\nYou may redistribute and modify this documentation under the terms of the CERN OHL\nv.1.2. (http://ohwr.org/cernohl). This documentation is distributed WITHOUT ANY EXPRESS\nOR IMPLIED WARRANTY, INCLUDING OF MERCHANTABILITY, SATISFACTORY QUALITY AND\nFITNESS FOR A PART"
- note added: "Note!\n\nThe sample PCB design included in this project is\nUNTESTED. Make sure it's correct before building\none or build the crossover on a protoboard for\nexample. The schematic should be correct since\nI built a crossover according to it."
Changed lines of the file:
@@
 Sheet 1 1
 Title "Two Way Speaker Crossover"
-Date "2019-11-30"
-Rev "A"
+Date "2020-01-07"
+Rev "B"
 Comp "Eero Talus"
-Comment1 "W-170S woofer and a SC-10N tweeter."
+Comment1 "W-170S woofer and a Visaton SC-10 N tweeter."
 Comment2 "Two way speaker crossover for a Visaton "
 Comment3 ""
@@
 F 3 "https://www.tme.eu/Document/27c0719e632264b7132c0e127fb04b62/ax20w.pdf" H 2150 1500 50  0001 C CNN
 F 4 "Royal Ohm PRW020JW82JB00" V 2150 1500 50  0001 C CNN "#"
+F 5 "20W" V 2150 1500 50  0000 C CNN "P"
 	1    2150 1500
 	0    -1   -1   0
@@
 F 0 "R4" V 2293 3300 50  0000 C CNN
 F 1 "4R7" V 2384 3300 50  0000 C CNN
-F 2 "Resistor_THT:R_Axial_Power_L60.0mm_W14.0mm_P66.04mm" V 2430 3300 50  0001 C CNN
+F 2 "etal_Resistors_THT:Resistor_Power_Axial_L91.5_W20.2_H20.2" V 2430 3300 50  0001 C CNN
 F 3 "https://www.tme.eu/Document/d2d66de62be8f045452af502fd3b634f/SR-Passives-CR-W.pdf" H 2500 3300 50  0001 C CNN
 F 4 "SR Passives CRL40W-4R7" V 2500 3300 50  0001 C CNN "#"
+F 5 "40W" V 2500 3300 50  0000 C CNN "P"
 	1    2500 3300
 	1    0    0    -1
@@
 F 3 "https://www.tme.eu/Document/27c0719e632264b7132c0e127fb04b62/ax20w.pdf" H 2600 1600 50  0001 C CNN
 F 4 "Royal Ohm PRW020JW82JB00" V 2600 1600 50  0001 C CNN "#"
+F 5 "20W" V 2600 1600 50  0000 C CNN "P"
 	1    2600 1600
 	-1   0    0    1
@@
 F 0 "R3" V 2093 2950 50  0000 C CNN
 F 1 "4R7" V 2184 2950 50  0000 C CNN
-F 2 "Resistor_THT:R_Axial_Power_L60.0mm_W14.0mm_P66.04mm" V 2230 2950 50  0001 C CNN
+F 2 "etal_Resistors_THT:Resistor_Power_Axial_L91.5_W20.2_H20.2" V 2230 2950 50  0001 C CNN
 F 3 "https://www.tme.eu/Document/d2d66de62be8f045452af502fd3b634f/SR-Passives-CR-W.pdf" H 2300 2950 50  0001 C CNN
 F 4 "SR Passives CRL40W-4R7" V 2300 2950 50  0001 C CNN "#"
+F 5 "40W" V 2300 2950 50  0000 C CNN "P"
 	1    2300 2950
 	0    1    1    0
@@
 Wire Wire Line
 	2500 2950 3150 2950
+Text Notes 7000 6500 0    50   ~ 0
+Copyright Eero Talus 2020.\n\nThis documentation describes Open Hardware and is licensed under the CERN OHL v. 1.2.\n\nYou may redistribute and modify this documentation under the terms of the CERN OHL\nv.1.2. (http://ohwr.org/cernohl). This documentation is distributed WITHOUT ANY EXPRESS\nOR IMPLIED WARRANTY, INCLUDING OF MERCHANTABILITY, SATISFACTORY QUALITY AND\nFITNESS FOR A PART
+Text Notes 4650 2500 0    157  ~ 0
+Note!\n\nThe sample PCB design included in this project is\nUNTESTED. Make sure it's correct before building\none or build the crossover on a protoboard for\nexample. The schematic should be correct since\nI built a crossover according to it.
 $EndSCHEMATC
